File: boards/CH/CH.kicad_sch (KiCad schematic)
At the start: 23 parts, among them K1 NRP-02-C-05DH, K2 NRP-02-C-05DH, K3 NRP-02-C-05DH, K4 NRP-02-C-05DH, K5 HF49FD/005-1H11, U1 6N137, U2 6N137, U3 КР293КП2Б, X1 BH-12 (2×6), X2 B5B-XH-A, X3 DG301-5.0-02P, X4 B4B-XH-A, X5 DG301-5.0-02P

Commit message: Платы PS, MC, CH, LR: расстановка, трассировка, 3D-модели посадочных мест
PS:
- разведена по расстановке из файла: +24V_IN 6 мм (участок у K1 — 4 мм),
  шина +24V 6 мм с отводами 3 мм, +5P 2 мм, остров U2 1,5 мм;
  заливка GND_P на B.Cu, вырез заливки под островом, вырезы ⌀8 у крепежа
- классы цепей в PS.kicad_pro: Default, Power5, Power24, Island
- U1: посадочное место под модуль XL4015E 54 × 24 × 15 на штырях
  (пятаки IN/OUT, 2 стойки М3) по чертежу продавца; переразведены
  OUT+ и отвод +24V к IN+

MC:
- X5 перенесён, переразведены KH, +5P, GND_P в этой зоне
- FU1: место под Bourns MF-R110 (корпус 8,9 × 3,0 × 14,0)

CH:
- K1…K5, X5: места исправлены по datasheet (NRP-02, HF49FD, JST VH),
  переразведены цепи реле

LR:
- плата перекомпонована: X5…X8 — B5B-XH-A, как X1…X4; группы M1…M4
  по одному образцу (индикатор, разъём, защита в два ряда);
  X1…X4, X9 и DD1 на нижней стороне
- контур 176 × 59, 6 отверстий М3; разведена: сигналы F.Cu,
  GND_L заливкой B.Cu
- scripts/gen_LR_pcb.py удалён: описывал прежнюю раскладку с клеммами

Схемы:
- CH: X5 — JST VH (таблица Tbl_X5_CH_VH); MC: X3 — B4B-XH-A
  (кнопка KH с индикатором); PS: X11 убран; LR: у X5…X8 место
  B5B-XH-A
- sch_common: генератор не перезаписывает файл, сохранённый KiCad,
  без --force

3D-модели (lib/3dmodels):
- упрощённые по чертежам datasheet: NRP-02, HF49FD, NRP-15 (корпус),
  JST B2P-VH, Mornsun/K-CUT URB2405YMD (U2), Talema DPO-3.0-22 (кольцо
  лежит), Bourns MF-R110
- из библиотеки KiCad: PinSocket 1×3, 1×4, 1×12, Phoenix MKDS-1,5-2
- docs/3D-модели.md — источники размеров и что сверить

База компонентов: E-083 — Bourns MF-R110 (Ihold 1,1 А), «Выбран»;
csv перевыгружены
Parts:
- removed X5: DG301-5.0-02P, manipulator:TB_DG301-5.0_2P_V, symbol manipulator:Tbl_X4_CH
- added X5: B2P-VH, manipulator:JST_VH_B2P-VH_V, symbol manipulator:Tbl_X5_CH_VH
Connections:
- net +24V_M: now also X5.1 (+24V_M)
- net +5P: now also U3.1 (A); no longer U3.4 (OUT)
- net GND_L: now also U3.6 (OUT); no longer U3.2 (K)
- net GND_P: now also X5.2 (GND_P)
- net at DA2.4 (IP+): no longer DA1.6 (OUT2)
- net at R3.2: now also U3.4 (OUT); no longer U3.1 (A)
- net at K5.1 (A1): now also U3.2 (K); no longer U3.6 (OUT)
- no-connect marks 0 -> 4
Other:
- note added: "+24V, +24V_M, +5P, GND_P (контакты 6, 10 разъёма X1, разъёмы X3, X5, выходы U1…DA1, K5); остров: +5V_L, 3V3,"
- note added: "7. Типы разъёмов X1…X5 в базе отсутствуют и показаны как предложение: X1 — IDC BH-12 (2 × 6) под ответную"
- note added: "9. Двигатель подключается проводами прямо к винтовым клеммникам модулей, мимо платы: OUT2 (DA1) → IP+ (DA2) —"
- note added: "GND_L (контакты 1, 2, 4, 12 разъёма X1, разъёмы X2, X4, светодиоды U1…U3, сигнальная часть DA2, R6, R7, C1)."
- note added: "перемычкой, IP− (DA2) → двигатель → OUT1 (DA1). Выводы OUT1, OUT2, IP+, IP− на плате не подключены; +24V_M и GND_P"
- note added: "подаются проводом с разъёма X5 (у K5) на клеммник POWER модуля DA1 и параллельно через VM, GND гребёнки."
- note added: "часть разъёмов X6…X9 платы MC; X2 — JST B5B-XH-A; X3 — клеммник DG301-5.0-02P; X4 — JST B4B-XH-A; X5 — JST B2P-VH."
- note removed: "+24V, +24V_M, +5P, GND_P (контакты 6, 10 разъёма X1, разъёмы X4, X5, выходы U1…DA1, K5); остров: +5V_L, 3V3,"
- note removed: "7. Типы разъёмов X1…X3, X5 в базе отсутствуют и показаны как предложение: X1 — IDC BH-12 (2 × 6) под ответную"
- note removed: "GND_L (контакты 1, 2, 4, 12 разъёма X1, разъёмы X2, X3, светодиоды U1…U3, сигнальная часть DA2, R6, R7, C1)."
- note removed: "часть разъёмов X6…X9 платы MC; X2 — JST B5B-XH-A; X3 — JST B4B-XH-A; X4, X5 — клеммники DG301-5.0-02P."

Commit message: Документы плат PS, MC, CH, LR; обозначения по схеме кафедры, наименования плат
- Документы плат PS, MC, CH, LR: перечень элементов, схема Э3, чертёж
  печатной платы, сборочный чертёж, спецификация (docs/<КОД>/)
- .gitignore: выпущенные документы docs/<КОД>/*.pdf хранятся в истории
- 3D-модели плат boards/<КОД>/<КОД>.step — исходные данные для проекций СБ
- Обозначения СМ7.02.ПП.ДД.00: ПЭ3, Э3, СБ — .00.00, плата печатная — .01.00,
  спецификация платы — .00.00 без аббревиатуры; правила в CLAUDE.md
- scripts/doc_titles.py: обозначения, наименования, подписи и основная надпись
  в одном месте; генераторы схем и плат берут их оттуда
- scripts/gen_pe3.py: перечень элементов ПЭ3 (А4, ГОСТ 2.701, 2.104)
- Наименования: «Манипулятор для лабораторных работ», платы питания,
  микроконтроллера, силовой части, режима ЛР (README, board-partition, генераторы)
- Схемы PS, MC, CH, LR перегенерированы: основная надпись из doc_titles,
  BaseID разъёмов E-092, E-096, E-097, E-098
- LR: X5…X8 — разъёмы к панели ЛР (E-098) вместо клемм E-051
- База компонентов: тип и допуск резисторов в наименовании, новые позиции
  E-096…E-098, E-051 исключена
- Платы: настройки вывода на печать; LR — дорожки и заливка зон
- Пояснительная записка курсового проекта обновлена
Connections:
- net at DA2.4 (IP+): now also DA1.6 (OUT2)
- net MOTOR-: now reaches DA2.5 (IP-)
- net MOTOR+: now reaches DA1.5 (OUT1)
Other:
- note removed: "+24V, +24V_M, +5P, GND_P (контакты 6, 10 разъёма X1, разъёмы X3, X5, выходы U1…DA1, K5); остров: +5V_L, 3V3,"
- note removed: "1. Плата канала привода CH изготавливается в 4 экземплярах (M1…M4) плюс один запасной; все экземпляры одинаковы."
- note removed: "2. Граница гальванической развязки проходит внутри U1, U2 (6N137), U3 (КР293КП2Б) и DA2 (ACS712), а также по"
- note removed: "3. Реле режима K1…K4: при обесточенных катушках управление звеном идёт с платы MC (контакты NC); при подаче"
- note removed: "4. U1, U2 (6N137): выход с открытым коллектором, подтяжки R4, R5 к +5P, выход инвертирующий (инверсия — в ПО);"
- note removed: "5 В со стороны панели ЛР ток составит 16 мА — предел для 6N137 (15 мА), номинал требует уточнения."
- note removed: "5. DA2 (ACS712-20A): 100 мВ/А, покой VCC/2 = 2,5 В, выход ратиометричен питанию. Делитель R6/R7 (10 к / 20 к)"
- note removed: "6. Нумерация выводов покупных модулей DA1, DA2 и реле K1…K5 условная, нумерация U3 — по ТУ; сверить по"
- note removed: "7. Типы разъёмов X1…X5 в базе отсутствуют и показаны как предложение: X1 — IDC BH-12 (2 × 6) под ответную"
- note removed: "8. Требует уточнения: диоды, шунтирующие катушки K1…K5, и конденсаторы 0,1 мкФ по питанию U1, U2 (рекомендация"
- note removed: "9. Двигатель подключается проводами прямо к винтовым клеммникам модулей, мимо платы: OUT2 (DA1) → IP+ (DA2) —"
- note removed: "C1 (100 нФ, E-095) стоит за R6: у ACS712 допустимая ёмкость нагрузки не более 10 нФ, поэтому прямо на выход"
- note removed: "GND_L (контакты 1, 2, 4, 12 разъёма X1, разъёмы X2, X4, светодиоды U1…U3, сигнальная часть DA2, R6, R7, C1)."
- note removed: "GND_P и GND_L на плате не соединять. +24V_M — питание двигателя после контакта реле K5."
- note removed: "datasheet 6N137) — таких позиций в базе компонентов нет."
- note removed: "Цепи IN1, IN2, RELE, CURR, SDA, SCL на плате MC имеют префикс канала (M1_IN1 и так далее)."
- note removed: "вывод 7 (VE) соединён с +5P, выводы 1 и 4 свободны. R1, R2 220 Ом дают 8,6 мА при 3,3 В; «Аккуратно!»: при"
- note removed: "датчика конденсатор не ставится. C1 снижает сопротивление источника для АЦП (6,7 кОм) и усредняет ШИМ:"
- note removed: "даёт 1,67 В покоя, 3,0 В при +20 А и 0,33 В при минус 20 А; при номинальном токе канала 1,2 А — 1,75 В."
- note removed: "и на плату не выводится: у платы Adafruit это 30 кОм (предел около 2 А), у клона номинал проверить —"
- note removed: "контактам реле K1…K4 (катушки — от шины KH относительно GND_P, контакты — в цепях острова). Силовая сторона:"
- note removed: "на 5 % смещает ноль на 1,25 А — нужна калибровка нуля в ПО при разомкнутом реле K5."
- note removed: "на канал, 640 мА на четыре канала — учесть при расчёте нагрузки +5P."
- note removed: "от него зависит пусковой ток двигателя (datasheet TI: R_ILIM не менее 15 кОм)."
- note removed: "перемычкой, IP− (DA2) → двигатель → OUT1 (DA1). Выводы OUT1, OUT2, IP+, IP− на плате не подключены; +24V_M и GND_P"
- note removed: "подаются проводом с разъёма X5 (у K5) на клеммник POWER модуля DA1 и параллельно через VM, GND гребёнки."
- note removed: "постоянная времени около 0,67 мс, полоса около 240 Гц. «Аккуратно!»: ноль привязан к +5V_L, уход питания"
- note removed: "часть разъёмов X6…X9 платы MC; X2 — JST B5B-XH-A; X3 — клеммник DG301-5.0-02P; X4 — JST B4B-XH-A; X5 — JST B2P-VH."
- note removed: "шелкографии и datasheet до разводки платы. Резистор ограничения тока ILIM распаян на самом модуле DA1"
- note removed: "шины KH (+5P, замкнута кнопкой режима на MC) — с панели ЛР (контакты NO). Ток катушек 4 × 40 мА = 160 мА"
- company: МГТУ им. Н.Э. Баумана, группа СМ7-21М -> МГТУ им. Н.Э. Баумана\n группа СМ7-21М
- title: Манипулятор учебный. Плата канала привода CH. Схема электрическая принципиальная -> Манипулятор для лабораторных работ.\nПлата силовой части.\nСхема электрическая принципиальная
