File: boards/LR/LR.kicad_sch (KiCad schematic)
At the start: 46 parts, among them X1 B5B-XH-A, X2 B5B-XH-A, X3 B5B-XH-A, X4 B5B-XH-A, X5 клеммы, X6 клеммы, X7 клеммы, X8 клеммы, X9 B4B-XH-A

Commit message: Платы PS, MC, CH, LR: расстановка, трассировка, 3D-модели посадочных мест
PS:
- разведена по расстановке из файла: +24V_IN 6 мм (участок у K1 — 4 мм),
  шина +24V 6 мм с отводами 3 мм, +5P 2 мм, остров U2 1,5 мм;
  заливка GND_P на B.Cu, вырез заливки под островом, вырезы ⌀8 у крепежа
- классы цепей в PS.kicad_pro: Default, Power5, Power24, Island
- U1: посадочное место под модуль XL4015E 54 × 24 × 15 на штырях
  (пятаки IN/OUT, 2 стойки М3) по чертежу продавца; переразведены
  OUT+ и отвод +24V к IN+

MC:
- X5 перенесён, переразведены KH, +5P, GND_P в этой зоне
- FU1: место под Bourns MF-R110 (корпус 8,9 × 3,0 × 14,0)

CH:
- K1…K5, X5: места исправлены по datasheet (NRP-02, HF49FD, JST VH),
  переразведены цепи реле

LR:
- плата перекомпонована: X5…X8 — B5B-XH-A, как X1…X4; группы M1…M4
  по одному образцу (индикатор, разъём, защита в два ряда);
  X1…X4, X9 и DD1 на нижней стороне
- контур 176 × 59, 6 отверстий М3; разведена: сигналы F.Cu,
  GND_L заливкой B.Cu
- scripts/gen_LR_pcb.py удалён: описывал прежнюю раскладку с клеммами

Схемы:
- CH: X5 — JST VH (таблица Tbl_X5_CH_VH); MC: X3 — B4B-XH-A
  (кнопка KH с индикатором); PS: X11 убран; LR: у X5…X8 место
  B5B-XH-A
- sch_common: генератор не перезаписывает файл, сохранённый KiCad,
  без --force

3D-модели (lib/3dmodels):
- упрощённые по чертежам datasheet: NRP-02, HF49FD, NRP-15 (корпус),
  JST B2P-VH, Mornsun/K-CUT URB2405YMD (U2), Talema DPO-3.0-22 (кольцо
  лежит), Bourns MF-R110
- из библиотеки KiCad: PinSocket 1×3, 1×4, 1×12, Phoenix MKDS-1,5-2
- docs/3D-модели.md — источники размеров и что сверить

База компонентов: E-083 — Bourns MF-R110 (Ihold 1,1 А), «Выбран»;
csv перевыгружены
Parts:
- X5, X6, X7, X8: footprint manipulator:TermGroup_5x_Banana4 -> manipulator:JST_XH_B5B-XH-A_L
Changed lines of the file:
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@@
 			)
 		)
-		(property "Footprint" "manipulator:TermGroup_5x_Banana4"
+		(property "Footprint" "manipulator:JST_XH_B5B-XH-A_L"
 			(at 223.52 25.4 0)
 			(hide yes)
@@
 			)
 		)
-		(property "Footprint" "manipulator:TermGroup_5x_Banana4"
+		(property "Footprint" "manipulator:JST_XH_B5B-XH-A_L"
 			(at 222.25 292.1 0)
 			(hide yes)
@@
 			)
 		)
-		(property "Footprint" "manipulator:TermGroup_5x_Banana4"
+		(property "Footprint" "manipulator:JST_XH_B5B-XH-A_L"
 			(at 222.25 114.3 0)
 			(hide yes)
@@
 			)
 		)
-		(property "Footprint" "manipulator:TermGroup_5x_Banana4"
+		(property "Footprint" "manipulator:JST_XH_B5B-XH-A_L"
 			(at 222.25 201.93 0)
 			(hide yes)

Commit message: Документы плат PS, MC, CH, LR; обозначения по схеме кафедры, наименования плат
- Документы плат PS, MC, CH, LR: перечень элементов, схема Э3, чертёж
  печатной платы, сборочный чертёж, спецификация (docs/<КОД>/)
- .gitignore: выпущенные документы docs/<КОД>/*.pdf хранятся в истории
- 3D-модели плат boards/<КОД>/<КОД>.step — исходные данные для проекций СБ
- Обозначения СМ7.02.ПП.ДД.00: ПЭ3, Э3, СБ — .00.00, плата печатная — .01.00,
  спецификация платы — .00.00 без аббревиатуры; правила в CLAUDE.md
- scripts/doc_titles.py: обозначения, наименования, подписи и основная надпись
  в одном месте; генераторы схем и плат берут их оттуда
- scripts/gen_pe3.py: перечень элементов ПЭ3 (А4, ГОСТ 2.701, 2.104)
- Наименования: «Манипулятор для лабораторных работ», платы питания,
  микроконтроллера, силовой части, режима ЛР (README, board-partition, генераторы)
- Схемы PS, MC, CH, LR перегенерированы: основная надпись из doc_titles,
  BaseID разъёмов E-092, E-096, E-097, E-098
- LR: X5…X8 — разъёмы к панели ЛР (E-098) вместо клемм E-051
- База компонентов: тип и допуск резисторов в наименовании, новые позиции
  E-096…E-098, E-051 исключена
- Платы: настройки вывода на печать; LR — дорожки и заливка зон
- Пояснительная записка курсового проекта обновлена
Parts:
- R1, R2, R3, R4: Note Последовательная защита линии SDA группы M1 со стороны клемм -> Последовательная защита линии SDA группы M1 со стороны пане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
- R5, R6, R7, R8: Note Последовательная защита линии SCL группы M1 со стороны клемм -> Последовательная защита линии SCL группы M1 со стороны пане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
- VD1, VD3, VD5, VD7: Note Встречный диод линии IN1 группы M1: ограничивает отрицательное напряжение с клеммы -> Встречный диод линии IN1 группы M1: ограничивает отрицательное напряжение со стороны панели
- VD2, VD4, VD6, VD8: Note Встречный диод линии IN2 группы M1: ограничивает отрицательное напряжение с клеммы -> Встречный диод линии IN2 группы M1: ограничивает отрицательное напряжение со стороны панели
- X1, X2, X3, X4: BaseID — -> E-098
- X5: value клеммы -> B5B-XH-A; BaseID E-051 -> E-098; Назначение Клеммы группы M1 (5 шт. E-051, винт + гнездо «банан» 4 мм):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 -> К панели ЛР, группа M1: 1 IN1, 2 IN2, 3 SDA, 4 SCL, 5 GND_L
- X6: value клеммы -> B5B-XH-A; BaseID E-051 -> E-098; Назначение Клеммы группы M2 (5 шт. E-051, винт + гнездо «банан» 4 мм):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 -> К панели ЛР, группа M2: 1 IN1, 2 IN2, 3 SDA, 4 SCL, 5 GND_L
- X7: value клеммы -> B5B-XH-A; BaseID E-051 -> E-098; Назначение Клеммы группы M3 (5 шт. E-051, винт + гнездо «банан» 4 мм):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 -> К панели ЛР, группа M3: 1 IN1, 2 IN2, 3 SDA, 4 SCL, 5 GND_L
- X8: value клеммы -> B5B-XH-A; BaseID E-051 -> E-098; Назначение Клеммы группы M4 (5 шт. E-051, винт + гнездо «банан» 4 мм):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 -> К панели ЛР, группа M4: 1 IN1, 2 IN2, 3 SDA, 4 SCL, 5 GND_L
Other:
- note added: "2. Защита каждой линии: панель — последовательный резистор 100 Ом (E-052) — ограничитель BAT54S (E-053) на 3,3 В"
- note added: "3. X5…X8 — разъёмы к панели ЛР (E-098), по одному на группу; к ним кабелем подключаются органы, в которые"
- note added: "IN1, IN2, SDA, SCL звена с платы MC на эту панель. В обычном режиме панель отключена от звена."
- note added: "студент включает свои провода. Тип этих органов на панели требует уточнения."
- note removed: "2. Защита каждой линии: клемма — последовательный резистор 100 Ом (E-052) — ограничитель BAT54S (E-053) на 3,3 В"
- note removed: "3. Клеммы X5…X8 — по 5 комбинированных приборных клемм E-051 на группу, 20 штук всего; каждый контакт таблицы —"
- note removed: "IN1, IN2, SDA, SCL звена с платы MC на клеммы этой панели. В обычном режиме клеммы отключены от звена."
- note removed: "отдельная клемма. Способ крепления (на плату или на переднюю стенку корпуса проводами) требует уточнения."
- company: МГТУ им. Н.Э. Баумана, группа СМ7-21М -> МГТУ им. Н.Э. Баумана\n группа СМ7-21М
- title: Манипулятор учебный. Плата панели лабораторных работ LR. Схема электрическая принципиальная -> Манипулятор для лабораторных работ.\nПлата режима ЛР.\nСхема электрическая принципиальная
Changed lines of the file:
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@@
 	(paper "A2")
 	(title_block
-		(title "Манипулятор учебный. Плата панели лабораторных работ LR. Схема электрическая принципиальная")
+		(title "Манипулятор для лабораторных работ.\\nПлата режима ЛР.\\nСхема электрическая принципиальная")
 		(date "2026-09-17")
 		(rev "LR-A1")
-		(company "МГТУ им. Н.Э. Баумана, группа СМ7-21М")
-		(comment 1 "--- Э3")
-		(comment 2 "Соловцов")
-		(comment 3 "---")
-		(comment 4 "---")
-		(comment 5 "---")
-		(comment 6 "Большаков")
+		(company "МГТУ им. Н.Э. Баумана\\n группа СМ7-21М")
+		(comment 1 "СМ7.02.04.00.00 Э3")
+		(comment 2 "Соловцов М.А.")
+		(comment 3 "Большаков А.А.")
 	)
 	(text "   Линии IN1, IN2 защищены встречным диодом 1N4148 (E-054): катод к линии, анод на GND_L."
@@
 		)
 	)
-	(text "2. Защита каждой линии: клемма — последовательный резистор 100 Ом (E-052) — ограничитель BAT54S (E-053) на 3,3 В"
+	(text "2. Защита каждой линии: панель — последовательный резистор 100 Ом (E-052) — ограничитель BAT54S (E-053) на 3,3 В"
 		(exclude_from_sim no)
 		(at -234.95 353.695 0)
@@
 		)
 	)
-	(text "   IN1, IN2, SDA, SCL звена с платы MC на клеммы этой панели. В обычном режиме клеммы отключены от звена."
+	(text "   IN1, IN2, SDA, SCL звена с платы MC на эту панель. В обычном режиме панель отключена от звена."
 		(exclude_from_sim no)
 		(at -234.95 349.25 0)
@@
 		)
 	)
-	(text "3. Клеммы X5…X8 — по 5 комбинированных приборных клемм E-051 на группу, 20 штук всего; каждый контакт таблицы —"
+	(text "3. X5…X8 — разъёмы к панели ЛР (E-098), по одному на группу; к ним кабелем подключаются органы, в которые"
 		(exclude_from_sim no)
 		(at -234.95 367.03 0)
@@
 		)
 	)
-	(text "   отдельная клемма. Способ крепления (на плату или на переднюю стенку корпуса проводами) требует уточнения."
+	(text "   студент включает свои провода. Тип этих органов на панели требует уточнения."
 		(exclude_from_sim no)
 		(at -234.95 371.475 0)
@@
 			)
 		)
-		(property "Note" "Последовательная защита линии SDA группы M1 со стороны клемм"
+		(property "Note" "Последовательная защита линии SDA группы M1 со стороны панели"
 			(at 177.8 138.43 0)
 			(hide yes)
@@
 			)
 		)
-		(property "Note" "Встречный диод линии IN2 группы M1: ограничивает отрицательное напряжение с клеммы"
+		(property "Note" "Встречный диод линии IN2 группы M1: ограничивает отрицательное напряжение со стороны панели"
 			(at 121.92 128.27 0)
 			(hide yes)
@@
 			)
 		)
-		(property "Value" "клеммы"
+		(property "Value" "B5B-XH-A"
 			(at 226.06 52.76 0)
 			(hide yes)
@@
 			)
 		)
-		(property "BaseID" "E-051"
+		(property "BaseID" "E-098"
 			(at 223.52 25.4 0)
 			(hide yes)
@@
 			)
 		)
-		(property "Назначение" "Клеммы группы M1 (5 шт. E-051, винт + гнездо «банан» 4 мм): 1 IN1, 2 IN2, 3 SDA, 4 SCL, 5 GND_L"
+		(property "Назначение" "К панели ЛР, группа M1: 1 IN1, 2 IN2, 3 SDA, 4 SCL, 5 GND_L"
 			(at 223.52 25.4 0)
 			(hide yes)
@@
 			)
 		)
-		(property "Note" "Последовательная защита линии SDA группы M1 со стороны клемм"
+		(property "Note" "Последовательная защита линии SDA группы M1 со стороны панели"
 			(at 177.8 316.23 0)
 			(hide yes)
@@
 			)
 		)
-		(property "Note" "Последовательная защита линии SCL группы M1 со стороны клемм"
+		(property "Note" "Последовательная защита линии SCL группы M1 со стороны панели"
 			(at 181.61 68.58 0)
 			(hide yes)
@@
 			)
 		)
-		(property "Value" "клеммы"
+		(property "Value" "B5B-XH-A"
 			(at 224.79 319.46 0)
 			(hide yes)
@@
 			)
 		)
-		(property "BaseID" "E-051"
+		(property "BaseID" "E-098"
 			(at 222.25 292.1 0)
 			(hide yes)
@@
 			)
 		)
-		(property "Назначение" "Клеммы группы M4 (5 шт. E-051, винт + гнездо «банан» 4 мм): 1 IN1, 2 IN2, 3 SDA, 4 SCL, 5 GND_L"
+		(property "Назначение" "К панели ЛР, группа M4: 1 IN1, 2 IN2, 3 SDA, 4 SCL, 5 GND_L"
 			(at 222.25 292.1 0)
 			(hide yes)
@@
 			)
 		)
-		(property "Note" "Встречный диод линии IN1 группы M1: ограничивает отрицательное напряжение с клеммы"
+		(property "Note" "Встречный диод линии IN1 группы M1: ограничивает отрицательное напряжение со стороны панели"
 			(at 121.92 283.21 0)
 			(hide yes)
@@
 			)
 		)
-		(property "Note" "Встречный диод линии IN1 группы M1: ограничивает отрицательное напряжение с клеммы"
+		(property "Note" "Встречный диод линии IN1 группы M1: ограничивает отрицательное напряжение со стороны панели"
 			(at 121.92 105.41 0)
 			(hide yes)
@@
 			)
 		)
-		(property "Note" "Встречный диод линии IN2 группы M1: ограничивает отрицательное напряжение с клеммы"
+		(property "Note" "Встречный диод линии IN2 группы M1: ограничивает отрицательное напряжение со стороны панели"
 			(at 123.19 39.37 0)
 			(hide yes)
@@
 			)
 		)
-		(property "BaseID" "—"
+		(property "BaseID" "E-098"
 			(at 67.31 201.93 0)
 			(hide yes)
@@
 			)
 		)
-		(property "Value" "клеммы"
+		(property "Value" "B5B-XH-A"
 			(at 224.79 141.66 0)
 			(hide yes)
@@
 			)
 		)
-		(property "BaseID" "E-051"
+		(property "BaseID" "E-098"
 			(at 222.25 114.3 0)
 			(hide yes)
@@
 			)
 		)
-		(property "Назначение" "Клеммы группы M2 (5 шт. E-051, винт + гнездо «банан» 4 мм): 1 IN1, 2 IN2, 3 SDA, 4 SCL, 5 GND_L"
+		(property "Назначение" "К панели ЛР, группа M2: 1 IN1, 2 IN2, 3 SDA, 4 SCL, 5 GND_L"
 			(at 222.25 114.3 0)
 			(hide yes)
@@
 			)
 		)
-		(property "Note" "Встречный диод линии IN1 группы M1: ограничивает отрицательное напряжение с клеммы"
+		(property "Note" "Встречный диод линии IN1 группы M1: ограничивает отрицательное напряжение со стороны панели"
 			(at 123.19 16.51 0)
 			(hide yes)
@@
 			)
 		)
-		(property "BaseID" "—"
+		(property "BaseID" "E-098"
 			(at 67.31 292.1 0)
 			(hide yes)
@@
 			)
 		)
-		(property "Note" "Последовательная защита линии SDA группы M1 со стороны клемм"
+		(property "Note" "Последовательная защита линии SDA группы M1 со стороны панели"
 			(at 177.8 226.06 0)
 			(hide yes)
@@
 			)
 		)
-		(property "Note" "Последовательная защита линии SDA группы M1 со стороны клемм"
+		(property "Note" "Последовательная защита линии SDA группы M1 со стороны панели"
 			(at 179.07 49.53 0)
 			(hide yes)
@@
 			)
 		)
-		(property "Note" "Последовательная защита линии SCL группы M1 со стороны клемм"
+		(property "Note" "Последовательная защита линии SCL группы M1 со стороны панели"
 			(at 180.34 245.11 0)
 			(hide yes)
@@
 			)
 		)
-		(property "Note" "Встречный диод линии IN2 группы M1: ограничивает отрицательное напряжение с клеммы"
+		(property "Note" "Встречный диод линии IN2 группы M1: ограничивает отрицательное напряжение со стороны панели"
 			(at 121.92 306.07 0)
 			(hide yes)
@@
 			)
 		)
-		(property "BaseID" "—"
+		(property "BaseID" "E-098"
 			(at 67.31 114.3 0)
 			(hide yes)
@@
 			)
 		)
-		(property "Note" "Последовательная защита линии SCL группы M1 со стороны клемм"
+		(property "Note" "Последовательная защита линии SCL группы M1 со стороны панели"
 			(at 180.34 157.48 0)
 			(hide yes)
@@
 			)
 		)
-		(property "Note" "Встречный диод линии IN2 группы M1: ограничивает отрицательное напряжение с клеммы"
+		(property "Note" "Встречный диод линии IN2 группы M1: ограничивает отрицательное напряжение со стороны панели"
 			(at 121.92 215.9 0)
 			(hide yes)
@@
 			)
 		)
-		(property "Note" "Последовательная защита линии SCL группы M1 со стороны клемм"
+		(property "Note" "Последовательная защита линии SCL группы M1 со стороны панели"
 			(at 180.34 335.28 0)
 			(hide yes)
@@
 			)
 		)
-		(property "Value" "клеммы"
+		(property "Value" "B5B-XH-A"
 			(at 224.79 229.29 0)
 			(hide yes)
@@
 			)
 		)
-		(property "BaseID" "E-051"
+		(property "BaseID" "E-098"
 			(at 222.25 201.93 0)
 			(hide yes)
@@
 			)
 		)
-		(property "Назначение" "Клеммы группы M3 (5 шт. E-051, винт + гнездо «банан» 4 мм): 1 IN1, 2 IN2, 3 SDA, 4 SCL, 5 GND_L"
+		(property "Назначение" "К панели ЛР, группа M3: 1 IN1, 2 IN2, 3 SDA, 4 SCL, 5 GND_L"
 			(at 222.25 201.93 0)
 			(hide yes)
@@
 			)
 		)
-		(property "Note" "Встречный диод линии IN1 группы M1: ограничивает отрицательное напряжение с клеммы"
+		(property "Note" "Встречный диод линии IN1 группы M1: ограничивает отрицательное напряжение со стороны панели"
 			(at 121.92 193.04 0)
 			(hide yes)
@@
 			)
 		)
-		(property "BaseID" "—"
+		(property "BaseID" "E-098"
 			(at 68.58 25.4 0)
 			(hide yes)
