File: boards/MC/MC.kicad_sch (KiCad schematic)
At the start: 23 parts, among them U1 CJMCU-9548, U2 КР293КП2Б, X1 B4B-XH-A, X10 B4B-XH-A, X2 B2P-VH, X3 B2B-XH-A, X4 B2B-XH-A, X5 B2P-VH, X6 BH-12 (2×6), X7 BH-12 (2×6), X8 BH-12 (2×6), X9 BH-12 (2×6)

Commit message: Схемы Э3: платы CH и LR, правки PS и MC
CH: схема канала привода (gen_CH_sch.py), оптроны в капсулах ГОСТ 2.730, X1 — вилка _D.
LR: схема панели (gen_LR_sch.py). PS: кнопка питания одним разъёмом X2 (B4B-XH-A:
контакт C–NO и индикатор 24 В), X12 убран, VD1 в линию с X1.1, примечания 5–6.
MC: узел U1 (КР293) под новое УГО, R5/R9, шина KH до R5. Сетка 1,27 у PS и LR.
check_sch.py: блоки «сетка 1,27» и «посадочные места».
Parts:
- removed U2: КР293КП2Б, manipulator:DIP-6_W7.62mm_H, symbol manipulator:OptoRelay_KR293
- added DD1: CJMCU-9548, manipulator:Module_CJMCU-9548, symbol manipulator:Module_TCA9548
- added R3: 10 кОм, manipulator:R_Axial_P10.16mm_V, symbol manipulator:R
- added R5: 20 кОм, manipulator:R_Axial_P10.16mm_V, symbol manipulator:R
- R4: renamed from R5; Note LED оптореле от шины KH (5 В), ≈8 мА -> LED оптореле от шины KH (5 В), около 8 мА
- U1: value CJMCU-9548 -> КР293КП2Б; footprint manipulator:Module_CJMCU-9548 -> manipulator:DIP-6_W7.62mm_H; symbol manipulator:Module_TCA9548 -> manipulator:OptoRelay_KR293; BaseID E-022 -> E-026; Note VCC 3,3 В; A2 — GND; A0/A1 — GPIO47/38; каналы 0–3 → M1…M4,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 -> Сигнал KH → ESP32: LED от шины KH через R5; ключ замыкает G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
- renumbered R4 to R1, R7 to R2, R3 to R6, R6 to R7, R1 to R8, R2 to R9, X3 to X2, X4 to X3, X5 to X4, X2 to X5, XS2 to XS1, XS1 to XS2
Connections:
- net 3V3: now also DD1.1 (VIN); no longer U1.1 (VIN)
- net GND_L: now also U1.6 (OUT), DD1.7 (A2), DD1.8 (GND), R5.1; no longer U1.7 (A2), U1.8 (GND)
- net GND_P: now also U1.2 (K)
- net KH: now also R4.1; no longer R4.2
- net M1_SCL: now also DD1.10 (SC0); no longer U1.10 (SC0)
- net M1_SDA: now also DD1.9 (SD0); no longer U1.9 (SD0)
- net M2_SCL: now also DD1.12 (SC1); no longer U1.12 (SC1)
- net M2_SDA: now also DD1.11 (SD1); no longer U1.11 (SD1)
- net M3_SCL: now also DD1.14 (SC2); no longer U1.14 (SC2)
- net M3_SDA: now also DD1.13 (SD2); no longer U1.13 (SD2)
- net M4_SCL: now also DD1.16 (SC3); no longer U1.16 (SC3)
- net M4_SDA: now also DD1.15 (SD3); no longer U1.15 (SD3)
- net MUX-A0: now also DD1.5 (A0); no longer U1.5 (A0)
- net MUX-A1: now also DD1.6 (A1); no longer U1.6 (A1)
- net MUX-RST: now also DD1.4 (RST); no longer U1.4 (RST)
- net at XS1.4 (IO1): now also R3.2, R5.2; no longer X1.3 (RX)
- net at R7.2, XS1.7 (IO41): now also U1.4 (OUT)
- net at R8.2, X10.3 (SDA), XS2.12 (IO8): now also DD1.2 (SDA); no longer U1.2 (SDA)
- net at R9.2, X10.2 (SCL), XS2.15 (IO9): now also DD1.3 (SCL); no longer U1.3 (SCL)
- new net: R4.2, U1.1 (A)
- new net: R3.1, X1.3 (RX)
Other:
- note added: "1. A1 — модуль YD-ESP32-S3 N16R8 (E-020) вставляется в гнёзда XS1 (ряд J1), XS2 (ряд J3). Выводы гнёзд сгруппированы по назначению,"
- note added: "номера контактов — по раскладке ESP32-S3-DevKitC-1 v1.1 (docs.espressif.com), контакт 1 — у разъёма USB; YD-ESP32-S3 — клон,"
- note added: "сверить с шелкографией. Питание модуля — +5V_L на вывод 5V; 3V3 — с модуля (E-011)."
- note removed: "1. A1 — модуль YD-ESP32-S3 N16R8 (E-020) вставляется в гнёзда XS1 (ряд J1), XS2 (ряд J3). Выводы гнёзд на схеме сгруппированы по назначению,"
- note removed: "2. GPIO (принятая распиновка, «Аккуратно!»): M1 IN1/IN2/CURR/RELE — 10/11/4/18; M2 — 12/13/5/21; M3 — 14/15/6/39; M4 — 16/17/7/40;"
- note removed: "3. Граница развязки: на +5P/GND_P — X2, кнопка KH (X3), шина KH с R4, светодиод U2 (через R5) и контакты 6, 8, 10 разъёмов X6…X9;"
- note removed: "4. Нумерация выводов U1 (модуль CJMCU-9548) и U2 (КР293КП2Б) — условная, сверить по шелкографии модуля и ТУ перед платой."
- note removed: "5. Шина KH (+5P, замкнута кнопкой) идёт на катушки реле режима плат CH; ESP32 читает состояние через U2 (вход инвертный)."
- note removed: "6. Разъёмы (типы — предложение, см. перечень элементов): X2, X5 — JST B2P-VH (E-019); X3, X4 — JST B2B-XH-A (E-018);"
- note removed: "7. E-073 (защита RX ESP32 от 5-вольтового передатчика схвата) — предложение, обвязка не определена: контроллер схвата не выбран."
- note removed: "A1 — модуль YD-ESP32-S3 N16R8 (E-020) в гнёздах XS1 (ряд J1), XS2 (ряд J3)"
- note removed: "SDA 8, SCL 9; MUX A0 47, A1 38, RST 42; KH 41; UART1 схвата RX 1 / TX 2; концевик M1 — 48 (предложение). ПК — родной USB (19/20)."
- note removed: "X1, X10 — JST B4B-XH-A (E-092); X6…X9 — IDC BH-12 (2 × 6, 2,54 мм); XS1, XS2 — гнездовые линейки PBS-22 (2,54 мм)."
- note removed: "Питание модуля — +5V_L на вывод 5V; 3V3 — с модуля (E-011)."
- note removed: "Резерв: 3, 43/44 (TX/RX). Не использовать: 0, 45, 46 (strapping), 35–37 (PSRAM). Проверить: на YD-ESP32-S3 GPIO48/38 могут быть"
- note removed: "всё остальное — остров (+5V_L, 3V3, GND_L). GND_P и GND_L на плате не соединять."
- note removed: "заняты бортовыми светодиодами (перемычки на модуле)."
- note removed: "номера контактов — по раскладке ESP32-S3-DevKitC-1 v1.1 (docs.espressif.com), контакт 1 — у разъёма USB; YD-ESP32-S3 — клон, сверить с шелкографией."
- moved on the sheet: C1, FU1, R1, R2, R4, R6, R7, R8, R9, X1, X10, X2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

Commit message: Платы PS, MC, CH, LR: расстановка, трассировка, 3D-модели посадочных мест
PS:
- разведена по расстановке из файла: +24V_IN 6 мм (участок у K1 — 4 мм),
  шина +24V 6 мм с отводами 3 мм, +5P 2 мм, остров U2 1,5 мм;
  заливка GND_P на B.Cu, вырез заливки под островом, вырезы ⌀8 у крепежа
- классы цепей в PS.kicad_pro: Default, Power5, Power24, Island
- U1: посадочное место под модуль XL4015E 54 × 24 × 15 на штырях
  (пятаки IN/OUT, 2 стойки М3) по чертежу продавца; переразведены
  OUT+ и отвод +24V к IN+

MC:
- X5 перенесён, переразведены KH, +5P, GND_P в этой зоне
- FU1: место под Bourns MF-R110 (корпус 8,9 × 3,0 × 14,0)

CH:
- K1…K5, X5: места исправлены по datasheet (NRP-02, HF49FD, JST VH),
  переразведены цепи реле

LR:
- плата перекомпонована: X5…X8 — B5B-XH-A, как X1…X4; группы M1…M4
  по одному образцу (индикатор, разъём, защита в два ряда);
  X1…X4, X9 и DD1 на нижней стороне
- контур 176 × 59, 6 отверстий М3; разведена: сигналы F.Cu,
  GND_L заливкой B.Cu
- scripts/gen_LR_pcb.py удалён: описывал прежнюю раскладку с клеммами

Схемы:
- CH: X5 — JST VH (таблица Tbl_X5_CH_VH); MC: X3 — B4B-XH-A
  (кнопка KH с индикатором); PS: X11 убран; LR: у X5…X8 место
  B5B-XH-A
- sch_common: генератор не перезаписывает файл, сохранённый KiCad,
  без --force

3D-модели (lib/3dmodels):
- упрощённые по чертежам datasheet: NRP-02, HF49FD, NRP-15 (корпус),
  JST B2P-VH, Mornsun/K-CUT URB2405YMD (U2), Talema DPO-3.0-22 (кольцо
  лежит), Bourns MF-R110
- из библиотеки KiCad: PinSocket 1×3, 1×4, 1×12, Phoenix MKDS-1,5-2
- docs/3D-модели.md — источники размеров и что сверить

База компонентов: E-083 — Bourns MF-R110 (Ihold 1,1 А), «Выбран»;
csv перевыгружены
Parts:
- X2: value B2B-XH-A -> B4B-XH-A; footprint manipulator:JST_XH_B2B-XH-A_L -> manipulator:JST_XH_B4B-XH-A_L
- X4, X5: value B2P-VH -> DG301-5.0-02P; footprint manipulator:JST_VH_B2P-VH_L -> manipulator:TB_DG301-5.0_2P_R
Connections:
- net GND_P: now also X2.4 (GND_P)
- net KH: now also X2.3 (KH)
Other:
- moved on the sheet: R1
Changed lines of the file:
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@@
 	)
 	(junction
+		(at 91.44 102.87)
+		(diameter 0)
+		(color 0 0 0 0)
+	)
+	(junction
 		(at 215.9 147.32)
 		(diameter 0)
@@
 	(wire
 		(pts
+			(xy 78.74 113.03) (xy 81.28 113.03)
+		)
+		(stroke
+			(width 0.3048)
+			(type default)
+		)
+	)
+	(wire
+		(pts
 			(xy 293.37 302.26) (xy 354.33 302.26)
 		)
@@
 	(wire
 		(pts
+			(xy 81.28 107.95) (xy 81.28 102.87)
+		)
+		(stroke
+			(width 0.3048)
+			(type default)
+		)
+	)
+	(wire
+		(pts
 			(xy 215.9 149.86) (xy 215.9 154.94)
 		)
@@
 	(wire
 		(pts
+			(xy 78.74 107.95) (xy 81.28 107.95)
+		)
+		(stroke
+			(width 0.3048)
+			(type default)
+		)
+	)
+	(wire
+		(pts
 			(xy 300.99 109.22) (xy 300.99 226.06)
 		)
@@
 	(wire
 		(pts
-			(xy 81.28 118.11) (xy 81.28 123.19)
+			(xy 91.44 118.11) (xy 91.44 123.19)
 		)
 		(stroke
@@
 	(wire
 		(pts
+			(xy 81.28 113.03) (xy 81.28 123.19)
+		)
+		(stroke
+			(width 0.3048)
+			(type default)
+		)
+	)
+	(wire
+		(pts
 			(xy 255.27 124.46) (xy 270.51 124.46)
 		)
@@
 			)
 		)
-		(property "Value" "B2P-VH"
+		(property "Value" "DG301-5.0-02P"
 			(at 36.83 192.46 0)
 			(hide yes)
@@
 			)
 		)
-		(property "Footprint" "manipulator:JST_VH_B2P-VH_L"
+		(property "Footprint" "manipulator:TB_DG301-5.0_2P_R"
 			(at 77.47 180.34 0)
 			(hide yes)
@@
 	)
 	(symbol
+		(lib_id "manipulator:GND_P")
+		(at 91.44 123.19 0)
+		(unit 1)
+		(body_style 1)
+		(exclude_from_sim no)
+		(in_bom yes)
+		(on_board yes)
+		(in_pos_files yes)
+		(dnp no)
+		(property "Reference" "#PWR076"
+			(at 83.82 119.38 0)
+			(hide yes)
+			(show_name no)
+			(do_not_autoplace no)
+			(effects
+				(font
+					(face "GOST 2.304")
+					(size 3.5 3.5)
+					(italic yes)
+				)
+			)
+		)
+		(property "Value" "GND_P"
+			(at 91.44 128.27 0)
+			(show_name no)
+			(do_not_autoplace no)
+			(effects
+				(font
+					(face "GOST 2.304")
+					(size 2.5 2.5)
+					(italic yes)
+				)
+			)
+		)
+		(property "Footprint" ""
+			(at 91.44 123.19 0)
+			(hide yes)
+			(show_name no)
+			(do_not_autoplace no)
+			(effects
+				(font
+					(face "GOST 2.304")
+					(size 2.5 2.5)
+					(italic yes)
+				)
+			)
+		)
+		(property "Datasheet" ""
+			(at 91.44 123.19 0)
+			(hide yes)
+			(show_name no)
+			(do_not_autoplace no)
+			(effects
+				(font
+					(face "GOST 2.304")
+					(size 2.5 2.5)
+					(italic yes)
+				)
+			)
+		)
+		(property "Description" ""
+			(at 91.44 123.19 0)
+			(hide yes)
+			(show_name no)
+			(do_not_autoplace no)
+			(effects
+				(font
+					(face "GOST 2.304")
+					(size 2.5 2.5)
+					(italic yes)
+				)
+			)
+		)
+		(pin "1"
+		)
+		(instances
+			(project "MC"
+				(path "/3c7e9a10-5b2d-4e8f-9a61-0d4c2b7f6e55"
+					(reference "#PWR076")
+					(unit 1)
+				)
+			)
+		)
+	)
+	(symbol
 		(lib_id "manipulator:3V3")
 		(at 271.78 38.1 0)
@@
 		(dnp no)
 		(property "Reference" "X2"
-			(at 38.354 109.474 0)
+			(at 38.354 119.63 0)
 			(show_name no)
 			(do_not_autoplace no)
@@
 			)
 		)
-		(property "Value" "B2B-XH-A"
+		(property "Value" "B4B-XH-A"
 			(at 35.56 109.91 0)
 			(hide yes)
@@
 			)
 		)
-		(property "Footprint" "manipulator:JST_XH_B2B-XH-A_L"
+		(property "Footprint" "manipulator:JST_XH_B4B-XH-A_L"
 			(at 76.2 97.79 0)
 			(hide yes)
@@
 		(pin "2"
 		)
+		(pin "3"
+		)
+		(pin "4"
+		)
 		(instances
 			(project "MC"
@@
 	(symbol
 		(lib_id "manipulator:R")
-		(at 81.28 110.49 0)
+		(at 91.44 110.49 0)
 		(unit 1)
 		(body_style 1)
@@
 		(dnp no)
 		(property "Reference" "R1"
-			(at 90.932 109.22 0)
+			(at 101.092 109.22 0)
 			(show_name no)
 			(do_not_autoplace no)
@@
 		)
 		(property "Value" "1 кОм"
-			(at 94.742 114.3 0)
+			(at 104.902 114.3 0)
 			(show_name no)
 			(do_not_autoplace no)
@@
 		)
 		(property "Footprint" "manipulator:R_Axial_P10.16mm_V"
-			(at 81.28 110.49 0)
+			(at 91.44 110.49 0)
 			(hide yes)
 			(show_name no)
@@
 		)
 		(property "Datasheet" ""
-			(at 81.28 110.49 0)
+			(at 91.44 110.49 0)
 			(hide yes)
 			(show_name no)
@@
 		)
 		(property "Description" ""
-			(at 81.28 110.49 0)
+			(at 91.44 110.49 0)
 			(hide yes)
 			(show_name no)
@@
 		)
 		(property "BaseID" "E-025"
-			(at 81.28 110.49 0)
+			(at 91.44 110.49 0)
 			(hide yes)
 			(show_name no)
@@
 		)
 		(property "Status" "Утверждено"
-			(at 81.28 110.49 0)
+			(at 91.44 110.49 0)
 			(hide yes)
 			(show_name no)
@@
 		)
 		(property "Note" "Подтяжка шины KH на GND_P"
-			(at 81.28 110.49 0)
+			(at 91.44 110.49 0)
 			(hide yes)
 			(show_name no)
@@
 			)
 		)
-		(property "Value" "B2P-VH"
+		(property "Value" "DG301-5.0-02P"
 			(at 36.83 225.48 0)
 			(hide yes)
@@
 			)
 		)
-		(property "Footprint" "manipulator:JST_VH_B2P-VH_L"
+		(property "Footprint" "manipulator:TB_DG301-5.0_2P_R"
 			(at 77.47 213.36 0)
 			(hide yes)

Commit message: Документы плат PS, MC, CH, LR; обозначения по схеме кафедры, наименования плат
- Документы плат PS, MC, CH, LR: перечень элементов, схема Э3, чертёж
  печатной платы, сборочный чертёж, спецификация (docs/<КОД>/)
- .gitignore: выпущенные документы docs/<КОД>/*.pdf хранятся в истории
- 3D-модели плат boards/<КОД>/<КОД>.step — исходные данные для проекций СБ
- Обозначения СМ7.02.ПП.ДД.00: ПЭ3, Э3, СБ — .00.00, плата печатная — .01.00,
  спецификация платы — .00.00 без аббревиатуры; правила в CLAUDE.md
- scripts/doc_titles.py: обозначения, наименования, подписи и основная надпись
  в одном месте; генераторы схем и плат берут их оттуда
- scripts/gen_pe3.py: перечень элементов ПЭ3 (А4, ГОСТ 2.701, 2.104)
- Наименования: «Манипулятор для лабораторных работ», платы питания,
  микроконтроллера, силовой части, режима ЛР (README, board-partition, генераторы)
- Схемы PS, MC, CH, LR перегенерированы: основная надпись из doc_titles,
  BaseID разъёмов E-092, E-096, E-097, E-098
- LR: X5…X8 — разъёмы к панели ЛР (E-098) вместо клемм E-051
- База компонентов: тип и допуск резисторов в наименовании, новые позиции
  E-096…E-098, E-051 исключена
- Платы: настройки вывода на печать; LR — дорожки и заливка зон
- Пояснительная записка курсового проекта обновлена
Parts:
- X2: BaseID E-018 -> E-092
- X6, X7, X8, X9: BaseID — -> E-096
- XS1, XS2: BaseID — -> E-097
Other:
- note added: "1. A1 — модуль YD-ESP32-S3 N16R8 (E-020) вставляется в гнёзда XS1, XS2. Выводы гнёзд сгруппированы по назначению,"
- note added: "контакт 1 — у разъёма USB; Питание модуля - +5V_L на вывод 5V; 3V3 - с модуля (E-011)."
- note removed: "1. A1 — модуль YD-ESP32-S3 N16R8 (E-020) вставляется в гнёзда XS1 (ряд J1), XS2 (ряд J3). Выводы гнёзд сгруппированы по назначению,"
- note removed: "номера контактов — по раскладке ESP32-S3-DevKitC-1 v1.1 (docs.espressif.com), контакт 1 — у разъёма USB; YD-ESP32-S3 — клон,"
- note removed: "сверить с шелкографией. Питание модуля — +5V_L на вывод 5V; 3V3 — с модуля (E-011)."
- company: МГТУ им. Н.Э. Баумана, группа СМ7-21М -> МГТУ им. Н.Э. Баумана \nгруппа СМ7-21М
- title: Манипулятор учебный. Плата контроллера MC. Схема электрическая принципиальная -> Манипулятор для лабораторных работ \nПлата микроконтроллера. \nСхема электрическая принципиальная
