File: boards/PS/PS.kicad_sch (KiCad schematic)
At the start: 20 parts, among them K1 NRP-15-C-24D, U1 Модуль XL4015E, U2 VRB2405YMD-10WR3, X1 DG301-5.0-02P-12, X10 DG301-5.0-02P-12, X11 B2B-XH-A, X2 B4B-XH-A, X3 B2P-VH, X4 B2P-VH, X5 B2B-XH-A, X6 DG301-5.0-02P-12, X7 DG301-5.0-02P-12, X8 DG301-5.0-02P-12, X9 DG301-5.0-02P-12

Commit message: Схемы Э3: платы CH и LR, правки PS и MC
CH: схема канала привода (gen_CH_sch.py), оптроны в капсулах ГОСТ 2.730, X1 — вилка _D.
LR: схема панели (gen_LR_sch.py). PS: кнопка питания одним разъёмом X2 (B4B-XH-A:
контакт C–NO и индикатор 24 В), X12 убран, VD1 в линию с X1.1, примечания 5–6.
MC: узел U1 (КР293) под новое УГО, R5/R9, шина KH до R5. Сетка 1,27 у PS и LR.
check_sch.py: блоки «сетка 1,27» и «посадочные места».
Parts:
- VD2: Status Предложение -> Утверждено
- X2: BaseID E-092 -> E-018; Назначение Кнопка питания E-002: 1 — катушка K1 (A2), 2 — GND_P (контакт кнопки замыкает 1–2); 3 — подсветка GND_P, 4 — подсветка +24V (после реле) -> Кнопка питания E-002: 1 — катушка K1 (A2), 2 — GND_P (контакт C–NO замыкает 1–2); 3 — GND_P, 4 — +24V после реле (встроенный индикатор 24 В)
- renumbered R2 to R1, X5 to X4, X4 to X5
Other:
- note added: "1. Вне платы: адаптер GST220A24-R7B (E-001) → гнездо KPJX-PM-4S (E-014) → предохранитель ATO 10 А (E-003) в проводе 18 AWG → X1."
- note added: "4. Фильтр +5P: L1 — Talema DPO-3.0-22 (E-012), C1 — 470 мкФ 16 В (E-093), C2 — 100 нФ X7R (E-094); f0 около 1,6 кГц."
- note added: "5. Подсветка кнопок — встроенные индикаторы 24 В, резисторов нет: кнопка питания E-002 — X2 (3, 4), кнопка KH E-024 — X11"
- note added: "6. Типы разъёмов (перечень элементов): X1, X6…X10 — DG301-5.0-02P-12 (E-017); X2 — JST B4B-XH-A, X5, X11 — B2B-XH-A (E-018);"
- note added: "7. K1: контакт 1C — 20 А при 28 В DC (datasheet NCR); NC (вывод 5) не используется. Перед пайкой прозвонить COM–NC обесточенного реле:"
- note added: "X3, X4 — B2P-VH (E-019)."
- note added: "Контакты гнезда: 1+2 — +24, 3+4 — GND, каждая пара параллельно (7,5 А/контакт при токе до 9,2 А); распайку сверить с datasheet R7B."
- note added: "кабелем к кнопке, минуя LR. Кнопка E-002 — с фиксацией (самоподхвата K1 нет). Индикатор «+5P есть» E-008 — на панели, R2 и X5."
- note added: "расположение выводов принято по виду снизу из datasheet."
- note removed: "1. Вне платы: адаптер GST220A24-R7B (E-001) → гнездо KPJX-PM-4S (E-014) → предохранитель ATO 10 А (E-003)"
- note removed: "4. Фильтр +5P: L1 — Talema DPO-3.0-22 (E-012), C1 — 470 мкФ 16 В (E-093), C2 — 100 нФ X7R (E-094); f₀ ≈ 1,6 кГц."
- note removed: "5. Подсветка кнопок — встроенные индикаторы 24 В, резисторов нет: кнопка питания E-002 — X2 (4: +24V, 3: GND_P),"
- note removed: "6. Типы разъёмов (см. перечень элементов): X1, X6…X10 — DG301-5.0-02P-12 (E-017); X2 — JST B4B-XH-A (E-092);"
- note removed: "7. K1: контакт 1C — 20 А при 28 В DC (datasheet NCR); NC (вывод 5) не используется. Перед пайкой прозвонить COM–NC"
- note removed: "8. Позиции с полем Status = Предложение ждут решения (VD2)."
- note removed: "X5, X11 — JST B2B-XH-A (E-018); X3, X4 — JST B2P-VH (E-019)."
- note removed: "в проводе 18 AWG → X1. Контакты гнезда: 1+2 — +24, 3+4 — GND, каждая пара параллельно (7,5 А/контакт"
- note removed: "кнопка KH E-024 — от X11 кабелем к кнопке (минуя LR). Индикатор «+5P есть» E-008 — на панели, на плате R2 и X5."
- note removed: "обесточенного реле и сверить с посадочным местом (расположение выводов принято по виду снизу из datasheet)."
- note removed: "при токе до 9,2 А); распайку сверить с datasheet штекера R7B адаптера."
- moved on the sheet: C1, C2, K1, L1, R1, U1, U2, VD1, VD2, X1, X10, X11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

Commit message: Платы PS, MC, CH, LR: расстановка, трассировка, 3D-модели посадочных мест
PS:
- разведена по расстановке из файла: +24V_IN 6 мм (участок у K1 — 4 мм),
  шина +24V 6 мм с отводами 3 мм, +5P 2 мм, остров U2 1,5 мм;
  заливка GND_P на B.Cu, вырез заливки под островом, вырезы ⌀8 у крепежа
- классы цепей в PS.kicad_pro: Default, Power5, Power24, Island
- U1: посадочное место под модуль XL4015E 54 × 24 × 15 на штырях
  (пятаки IN/OUT, 2 стойки М3) по чертежу продавца; переразведены
  OUT+ и отвод +24V к IN+

MC:
- X5 перенесён, переразведены KH, +5P, GND_P в этой зоне
- FU1: место под Bourns MF-R110 (корпус 8,9 × 3,0 × 14,0)

CH:
- K1…K5, X5: места исправлены по datasheet (NRP-02, HF49FD, JST VH),
  переразведены цепи реле

LR:
- плата перекомпонована: X5…X8 — B5B-XH-A, как X1…X4; группы M1…M4
  по одному образцу (индикатор, разъём, защита в два ряда);
  X1…X4, X9 и DD1 на нижней стороне
- контур 176 × 59, 6 отверстий М3; разведена: сигналы F.Cu,
  GND_L заливкой B.Cu
- scripts/gen_LR_pcb.py удалён: описывал прежнюю раскладку с клеммами

Схемы:
- CH: X5 — JST VH (таблица Tbl_X5_CH_VH); MC: X3 — B4B-XH-A
  (кнопка KH с индикатором); PS: X11 убран; LR: у X5…X8 место
  B5B-XH-A
- sch_common: генератор не перезаписывает файл, сохранённый KiCad,
  без --force

3D-модели (lib/3dmodels):
- упрощённые по чертежам datasheet: NRP-02, HF49FD, NRP-15 (корпус),
  JST B2P-VH, Mornsun/K-CUT URB2405YMD (U2), Talema DPO-3.0-22 (кольцо
  лежит), Bourns MF-R110
- из библиотеки KiCad: PinSocket 1×3, 1×4, 1×12, Phoenix MKDS-1,5-2
- docs/3D-модели.md — источники размеров и что сверить

База компонентов: E-083 — Bourns MF-R110 (Ihold 1,1 А), «Выбран»;
csv перевыгружены
Parts:
- removed X11: B2B-XH-A, manipulator:JST_XH_B2B-XH-A, symbol manipulator:Tbl_X11_PS
- X2: Назначение Кнопка питания E-002: 1 — катушка K1 (A2), 2 — GND_P (конта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 -> Кнопка питания E-002, контакт: 1 — катушка K1 (A2), 2 — GND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
- renumbered R1 to R2, X5 to X4, X4 to X5
Other:
- note added: "5. Подсветка кнопок — встроенные индикаторы 24 В, резисторов нет: кнопка питания E-002 — от X12, кнопка KH E-024 — от X11"
- note added: "6. Типы разъёмов (перечень элементов): X1, X6…X10 — DG301-5.0-02P-12 (E-017); X2, X5, X11, X12 — JST B2B-XH-A (E-018);"
- note added: "кабелем к кнопке, минуя LR. Индикатор «+5P есть» E-008 — на панели, на плате R2 и X5."
- note removed: "5. Подсветка кнопок — встроенные индикаторы 24 В, резисторов нет: кнопка питания E-002 — X2 (3, 4), кнопка KH E-024 — X11"
- note removed: "6. Типы разъёмов (перечень элементов): X1, X6…X10 — DG301-5.0-02P-12 (E-017); X2 — JST B4B-XH-A, X5, X11 — B2B-XH-A (E-018);"
- note removed: "кабелем к кнопке, минуя LR. Кнопка E-002 — с фиксацией (самоподхвата K1 нет). Индикатор «+5P есть» E-008 — на панели, R2 и X5."
- moved on the sheet: C1, C2, K1, L1, R2, U1, U2, VD1, VD2, X1, X10, X2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

Commit message: Документы плат PS, MC, CH, LR; обозначения по схеме кафедры, наименования плат
- Документы плат PS, MC, CH, LR: перечень элементов, схема Э3, чертёж
  печатной платы, сборочный чертёж, спецификация (docs/<КОД>/)
- .gitignore: выпущенные документы docs/<КОД>/*.pdf хранятся в истории
- 3D-модели плат boards/<КОД>/<КОД>.step — исходные данные для проекций СБ
- Обозначения СМ7.02.ПП.ДД.00: ПЭ3, Э3, СБ — .00.00, плата печатная — .01.00,
  спецификация платы — .00.00 без аббревиатуры; правила в CLAUDE.md
- scripts/doc_titles.py: обозначения, наименования, подписи и основная надпись
  в одном месте; генераторы схем и плат берут их оттуда
- scripts/gen_pe3.py: перечень элементов ПЭ3 (А4, ГОСТ 2.701, 2.104)
- Наименования: «Манипулятор для лабораторных работ», платы питания,
  микроконтроллера, силовой части, режима ЛР (README, board-partition, генераторы)
- Схемы PS, MC, CH, LR перегенерированы: основная надпись из doc_titles,
  BaseID разъёмов E-092, E-096, E-097, E-098
- LR: X5…X8 — разъёмы к панели ЛР (E-098) вместо клемм E-051
- База компонентов: тип и допуск резисторов в наименовании, новые позиции
  E-096…E-098, E-051 исключена
- Платы: настройки вывода на печать; LR — дорожки и заливка зон
- Пояснительная записка курсового проекта обновлена
Parts:
- X2: BaseID E-018 -> E-092
Other:
- note removed: "1. Вне платы: адаптер GST220A24-R7B (E-001) → гнездо KPJX-PM-4S (E-014) → предохранитель ATO 10 А (E-003) в проводе 18 AWG → X1."
- note removed: "2. Граница гальванической развязки — U2: цепи GND_P и GND_L на плате не соединять."
- note removed: "3. Выходы +24: X6…X9 — платы каналов CH1…CH4, X10 — схват; провод 20–22 AWG (E-081)."
- note removed: "4. Фильтр +5P: L1 — Talema DPO-3.0-22 (E-012), C1 — 470 мкФ 16 В (E-093), C2 — 100 нФ X7R (E-094); f0 около 1,6 кГц."
- note removed: "5. Подсветка кнопок — встроенные индикаторы 24 В, резисторов нет: кнопка питания E-002 — от X12, кнопка KH E-024 — от X11"
- note removed: "6. Типы разъёмов (перечень элементов): X1, X6…X10 — DG301-5.0-02P-12 (E-017); X2, X5, X11, X12 — JST B2B-XH-A (E-018);"
- note removed: "7. K1: контакт 1C — 20 А при 28 В DC (datasheet NCR); NC (вывод 5) не используется. Перед пайкой прозвонить COM–NC обесточенного реле:"
- note removed: "X3, X4 — B2P-VH (E-019)."
- note removed: "Контакты гнезда: 1+2 — +24, 3+4 — GND, каждая пара параллельно (7,5 А/контакт при токе до 9,2 А); распайку сверить с datasheet R7B."
- note removed: "кабелем к кнопке, минуя LR. Индикатор «+5P есть» E-008 — на панели, на плате R2 и X5."
- note removed: "расположение выводов принято по виду снизу из datasheet."
- company: МГТУ им. Н.Э. Баумана, группа СМ7-21М -> МГТУ им. Н.Э. Баумана\n группа СМ7-21М
- title: Манипулятор учебный. Плата питания PS. Схема электрическая принципиальная -> Манипулятор для лабораторных работ.\n Плата питания.\n Схема электрическая принципиальная
Changed lines of the file:
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@@
 	(paper "A3")
 	(title_block
-		(title "Манипулятор учебный. Плата питания PS. Схема электрическая принципиальная")
+		(title "Манипулятор для лабораторных работ.\\n Плата питания.\\n Схема электрическая принципиальная")
 		(date "2026-09-17")
 		(rev "PS-A1")
-		(company "МГТУ им. Н.Э. Баумана, группа СМ7-21М")
-		(comment 1 "--- Э3")
-		(comment 2 "Соловцов")
-		(comment 3 "---")
-		(comment 4 "---")
-		(comment 5 "---")
-		(comment 6 "Большаков")
-	)
-	(text "6. Типы разъёмов (перечень элементов): X1, X6…X10 — DG301-5.0-02P-12 (E-017); X2, X5, X11, X12 — JST B2B-XH-A (E-018);"
-		(exclude_from_sim no)
-		(at -289.814 209.042 0)
-		(effects
-			(font
-				(face "GOST 2.304")
-				(size 2.5 2.5)
-				(italic yes)
-			)
-			(justify left bottom)
-		)
-	)
-	(text "1. Вне платы: адаптер GST220A24-R7B (E-001) → гнездо KPJX-PM-4S (E-014) → предохранитель ATO 10 А (E-003) в проводе 18 AWG → X1."
-		(exclude_from_sim no)
-		(at -289.814 177.927 0)
-		(effects
-			(font
-				(face "GOST 2.304")
-				(size 2.5 2.5)
-				(italic yes)
-			)
-			(justify left bottom)
-		)
-	)
-	(text "4. Фильтр +5P: L1 — Talema DPO-3.0-22 (E-012), C1 — 470 мкФ 16 В (E-093), C2 — 100 нФ X7R (E-094); f0 около 1,6 кГц."
-		(exclude_from_sim no)
-		(at -289.814 195.707 0)
-		(effects
-			(font
-				(face "GOST 2.304")
-				(size 2.5 2.5)
-				(italic yes)
-			)
-			(justify left bottom)
-		)
-	)
-	(text "2. Граница гальванической развязки — U2: цепи GND_P и GND_L на плате не соединять."
-		(exclude_from_sim no)
-		(at -289.814 186.817 0)
-		(effects
-			(font
-				(face "GOST 2.304")
-				(size 2.5 2.5)
-				(italic yes)
-			)
-			(justify left bottom)
-		)
-	)
-	(text "   кабелем к кнопке, минуя LR. Индикатор «+5P есть» E-008 — на панели, на плате R2 и X5."
-		(exclude_from_sim no)
-		(at -289.814 204.597 0)
-		(effects
-			(font
-				(face "GOST 2.304")
-				(size 2.5 2.5)
-				(italic yes)
-			)
-			(justify left bottom)
-		)
-	)
-	(text "   Контакты гнезда: 1+2 — +24, 3+4 — GND, каждая пара параллельно (7,5 А/контакт при токе до 9,2 А); распайку сверить с datasheet R7B."
-		(exclude_from_sim no)
-		(at -289.814 182.372 0)
-		(effects
-			(font
-				(face "GOST 2.304")
-				(size 2.5 2.5)
-				(italic yes)
-			)
-			(justify left bottom)
-		)
-	)
-	(text "5. Подсветка кнопок — встроенные индикаторы 24 В, резисторов нет: кнопка питания E-002 — от X12, кнопка KH E-024 — от X11"
-		(exclude_from_sim no)
-		(at -289.814 200.152 0)
-		(effects
-			(font
-				(face "GOST 2.304")
-				(size 2.5 2.5)
-				(italic yes)
-			)
-			(justify left bottom)
-		)
-	)
-	(text "   расположение выводов принято по виду снизу из datasheet."
-		(exclude_from_sim no)
-		(at -289.814 222.377 0)
-		(effects
-			(font
-				(face "GOST 2.304")
-				(size 2.5 2.5)
-				(italic yes)
-			)
-			(justify left bottom)
-		)
-	)
-	(text "7. K1: контакт 1C — 20 А при 28 В DC (datasheet NCR); NC (вывод 5) не используется. Перед пайкой прозвонить COM–NC обесточенного реле:"
-		(exclude_from_sim no)
-		(at -289.814 217.932 0)
-		(effects
-			(font
-				(face "GOST 2.304")
-				(size 2.5 2.5)
-				(italic yes)
-			)
-			(justify left bottom)
-		)
-	)
-	(text "   X3, X4 — B2P-VH (E-019)."
-		(exclude_from_sim no)
-		(at -289.814 213.487 0)
-		(effects
-			(font
-				(face "GOST 2.304")
-				(size 2.5 2.5)
-				(italic yes)
-			)
-			(justify left bottom)
-		)
-	)
-	(text "3. Выходы +24: X6…X9 — платы каналов CH1…CH4, X10 — схват; провод 20–22 AWG (E-081)."
-		(exclude_from_sim no)
-		(at -289.814 191.262 0)
-		(effects
-			(font
-				(face "GOST 2.304")
-				(size 2.5 2.5)
-				(italic yes)
-			)
-			(justify left bottom)
-		)
+		(company "МГТУ им. Н.Э. Баумана\\n группа СМ7-21М")
+		(comment 1 "СМ7.02.01.00.00 Э3")
+		(comment 2 "Соловцов М.А.")
+		(comment 3 "Большаков А.А.")
 	)
 	(junction
@@
 			)
 		)
-		(property "BaseID" "E-018"
+		(property "BaseID" "E-092"
 			(at 180.34 66.04 0)
 			(hide yes)
